File: ES920LRB-Arduino-Shield/ES920LRB-Arduino-Shield.sch (KiCad schematic (older format))
At the start: 31 parts, among them J1 Conn_01x10_Female, J2 Conn_01x12_Female, M1 ES920LR2B, P1 Power, P2 Analog, P3 Digital, P4 Digital, P5 CONN_01X01, P6 CONN_01X01, P7 CONN_01X01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

Commit message: add arduino uno sheild pcb
add arduino uno sheild pcb
Parts:
- added JP5, JP6: SolderJumper_2_Open, Jumper:SolderJumper-2_P1.3mm_Open_Pad1.0x1.5mm, symbol Jumper:SolderJumper_2_Open
Connections:
- net 2: now also JP5.2 (B)
- net 3(**): now also JP6.2 (B)
- net at JP3.1 (A), Q3.3 (D), R8.2: now also JP5.1 (A)
- net at JP4.1 (A), Q4.3 (D), R7.2: now also JP6.1 (A)
Other:
- note added: "close"
- note added: "open"
- moved on the sheet: JP3
Changed lines of the file:
@@
 encoding utf-8
 Sheet 1 1
-Title "ES920LRB-Arduino-Shield"
+Title "ES920LRB-Arduino_Uno-Shield"
 Date "2021-11-24"
-Rev "1.4"
+Rev "1.6"
 Comp "teTra Aviation Corp."
 Comment1 ""
@@
 Reset
 $Comp
-L power:+3.3V #PWR01
-U 1 1 56D70538
-P 9150 1450
-F 0 "#PWR01" H 9150 1300 50  0001 C CNN
-F 1 "+3.3V" V 9150 1700 50  0000 C CNN
-F 2 "" H 9150 1450 50  0000 C CNN
-F 3 "" H 9150 1450 50  0000 C CNN
-	1    9150 1450
-	1    0    0    -1
-$EndComp
-$Comp
 L power:+5V #PWR02
 U 1 1 56D707BB
@@
 	1    0    0    -1
 $EndComp
-$Comp
-L power:+3V3 #PWR0103
-U 1 1 6193CC91
-P 1300 1650
-F 0 "#PWR0103" H 1300 1500 50  0001 C CNN
-F 1 "+3V3" H 1315 1823 50  0000 C CNN
-F 2 "" H 1300 1650 50  0001 C CNN
-F 3 "" H 1300 1650 50  0001 C CNN
-	1    1300 1650
-	1    0    0    -1
-$EndComp
 Wire Wire Line
 	5750 2150 5750 2500
@@
 L Jumper:SolderJumper_2_Open JP3
 U 1 1 619A575C
-P 8900 5400
-F 0 "JP3" H 8900 5605 50  0000 C CNN
-F 1 "SolderJumper_2_Open" H 8900 5514 50  0000 C CNN
-F 2 "Jumper:SolderJumper-2_P1.3mm_Open_Pad1.0x1.5mm" H 8900 5400 50  0001 C CNN
-F 3 "~" H 8900 5400 50  0001 C CNN
-	1    8900 5400
+P 8900 5250
+F 0 "JP3" H 8900 5455 50  0000 C CNN
+F 1 "SolderJumper_2_Open" H 8900 5364 50  0000 C CNN
+F 2 "Jumper:SolderJumper-2_P1.3mm_Open_Pad1.0x1.5mm" H 8900 5250 50  0001 C CNN
+F 3 "~" H 8900 5250 50  0001 C CNN
+	1    8900 5250
 	1    0    0    -1
 $EndComp
@@
 	1    0    0    -1
 $EndComp
-$Comp
-L power:+3V3 #PWR05
-U 1 1 61E7E904
-P 6200 3200
-F 0 "#PWR05" H 6200 3050 50  0001 C CNN
-F 1 "+3V3" H 6215 3373 50  0000 C CNN
-F 2 "" H 6200 3200 50  0001 C CNN
-F 3 "" H 6200 3200 50  0001 C CNN
-	1    6200 3200
-	1    0    0    -1
-$EndComp
 Wire Wire Line
 	4650 4100 4650 2350
@@
 	1700 2150 2300 2150
 $Comp
-L power:+5V #PWR06
-U 1 1 62099DDA
-P 7250 3200
-F 0 "#PWR06" H 7250 3050 50  0001 C CNN
-F 1 "+5V" H 7265 3373 50  0000 C CNN
-F 2 "" H 7250 3200 50  0001 C CNN
-F 3 "" H 7250 3200 50  0001 C CNN
-	1    7250 3200
-	1    0    0    -1
-$EndComp
-$Comp
 L Device:R R9
 U 1 1 620AFA4D
@@
 	7500 3300 7750 3300
 Wire Wire Line
-	8750 5400 7500 5400
-Wire Wire Line
 	7050 6050 7250 6050
 Wire Wire Line
@@
 Connection ~ 7250 6050
 Wire Wire Line
-	7250 6050 8750 6050
+	7250 6050 8400 6050
 Wire Wire Line
 	7500 3800 7500 5400
@@
 Text Label 9600 6050 0    60   ~ 0
 1(Tx)
-Text Label 9600 5400 0    60   ~ 0
+Text Label 9600 5250 0    60   ~ 0
 0(Rx)
 Wire Wire Line
@@
 	9600 4750 9050 4750
 Wire Wire Line
-	9050 5400 9600 5400
-Wire Wire Line
-	9600 6050 9050 6050
-Wire Wire Line
 	4650 4100 5450 4100
 Wire Wire Line
@@
 Wire Wire Line
 	2050 6050 6200 6050
+$Comp
+L power:+3.3V #PWR01
+U 1 1 56D70538
+P 9150 1450
+F 0 "#PWR01" H 9150 1300 50  0001 C CNN
+F 1 "+3.3V" V 9150 1700 50  0000 C CNN
+F 2 "" H 9150 1450 50  0000 C CNN
+F 3 "" H 9150 1450 50  0000 C CNN
+	1    9150 1450
+	1    0    0    -1
+$EndComp
+$Comp
+L power:+3.3V #PWR0103
+U 1 1 6228A2D0
+P 1300 1650
+F 0 "#PWR0103" H 1300 1500 50  0001 C CNN
+F 1 "+3.3V" V 1300 1900 50  0000 C CNN
+F 2 "" H 1300 1650 50  0000 C CNN
+F 3 "" H 1300 1650 50  0000 C CNN
+	1    1300 1650
+	1    0    0    -1
+$EndComp
+$Comp
+L power:+3.3V #PWR0104
+U 1 1 622A2386
+P 6200 3200
+F 0 "#PWR0104" H 6200 3050 50  0001 C CNN
+F 1 "+3.3V" V 6200 3450 50  0000 C CNN
+F 2 "" H 6200 3200 50  0000 C CNN
+F 3 "" H 6200 3200 50  0000 C CNN
+	1    6200 3200
+	1    0    0    -1
+$EndComp
+$Comp
+L power:+5V #PWR0105
+U 1 1 622BF7A1
+P 7250 3200
+F 0 "#PWR0105" H 7250 3050 50  0001 C CNN
+F 1 "+5V" V 7250 3400 50  0000 C CNN
+F 2 "" H 7250 3200 50  0000 C CNN
+F 3 "" H 7250 3200 50  0000 C CNN
+	1    7250 3200
+	1    0    0    -1
+$EndComp
+Text Notes 8800 4250 0    50   ~ 0
+close
+Text Notes 8800 5400 0    50   ~ 0
+open
+Text Notes 8800 6200 0    50   ~ 0
+open
+Text Notes 8800 4900 0    50   ~ 0
+open
+Text Label 9600 5650 0    60   ~ 0
+2
+Text Label 9600 6450 0    60   ~ 0
+3(**)
+$Comp
+L Jumper:SolderJumper_2_Open JP5
+U 1 1 623232ED
+P 8900 5650
+F 0 "JP5" H 8900 5855 50  0000 C CNN
+F 1 "SolderJumper_2_Open" H 8900 5764 50  0000 C CNN
+F 2 "Jumper:SolderJumper-2_P1.3mm_Open_Pad1.0x1.5mm" H 8900 5650 50  0001 C CNN
+F 3 "~" H 8900 5650 50  0001 C CNN
+	1    8900 5650
+	1    0    0    -1
+$EndComp
+Text Notes 8800 5800 0    50   ~ 0
+close
+$Comp
+L Jumper:SolderJumper_2_Open JP6
+U 1 1 6232A219
+P 8900 6450
+F 0 "JP6" H 8900 6655 50  0000 C CNN
+F 1 "SolderJumper_2_Open" H 8900 6564 50  0000 C CNN
+F 2 "Jumper:SolderJumper-2_P1.3mm_Open_Pad1.0x1.5mm" H 8900 6450 50  0001 C CNN
+F 3 "~" H 8900 6450 50  0001 C CNN
+	1    8900 6450
+	1    0    0    -1
+$EndComp
+Text Notes 8800 6600 0    50   ~ 0
+close
+Wire Wire Line
+	9050 5250 9600 5250
+Wire Wire Line
+	8750 6450 8400 6450
+Wire Wire Line
+	8400 6450 8400 6050
+Connection ~ 8400 6050
+Wire Wire Line
+	8400 6050 8750 6050
+Wire Wire Line
+	9050 6050 9600 6050
+Wire Wire Line
+	9050 5650 9600 5650
+Wire Wire Line
+	9050 6450 9600 6450
+Wire Wire Line
+	8750 5250 8400 5250
+Wire Wire Line
+	8400 5250 8400 5400
+Connection ~ 8400 5400
+Wire Wire Line
+	8400 5400 7500 5400
+Wire Wire Line
+	8400 5400 8400 5650
+Wire Wire Line
+	8400 5650 8750 5650
 $EndSCHEMATC
