File: ES920LRB-Arduino-Shield/ES920LRB-Arduino-Shield.kicad_pcb (KiCad board)
At the start: 2 copper layers, 68.6 x 53.3 mm, 18 parts, among them J1 Conn_01x10_Female, J2 Conn_01x12_Female, M1 ES920LR2B, P1 Power, P2 Analog, P3 Digital, P4 Digital, P5 CONN_01X01, P6 CONN_01X01, P7 CONN_01X01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

Commit message: add schematica v1.3
add schematica v1.3
Parts:
- added C1: 10uF, Capacitor_THT:C_Rect_L4.0mm_W2.5mm_P2.50mm, F.Cu at (201.5, 84.4)
- added JP4: SolderJumper_2_Open, Jumper:SolderJumper-2_P1.3mm_Open_Pad1.0x1.5mm, F.Cu at (192.0, 109.9)
- added L1: Logo, teTra:teTra-logo, F.Cu at (192.7, 81.9)
- added Q1: BSS138, Package_TO_SOT_SMD:SOT-23, F.Cu at (202.1, 88.7)
- added Q2: BSS138, Package_TO_SOT_SMD:SOT-23, F.Cu at (212.5, 80.6)
- added Q3: BSS138, Package_TO_SOT_SMD:SOT-23, F.Cu at (207.8, 84.6)
- added Q4: BSS138, Package_TO_SOT_SMD:SOT-23, F.Cu at (212.2, 85.1)
- added R10: 10k, Resistor_THT:R_Axial_DIN0207_L6.3mm_D2.5mm_P2.54mm_Vertical, F.Cu at (195.8, 89.4)
- added R4: 10k, Resistor_THT:R_Axial_DIN0207_L6.3mm_D2.5mm_P2.54mm_Vertical, F.Cu at (189.7, 85.3)
- added R6: 10k, Resistor_THT:R_Axial_DIN0207_L6.3mm_D2.5mm_P2.54mm_Vertical, F.Cu at (200.0, 80.3)
- added R7: 10k, Resistor_THT:R_Axial_DIN0207_L6.3mm_D2.5mm_P2.54mm_Vertical, F.Cu at (189.7, 89.4)
- added R8: 10k, Resistor_THT:R_Axial_DIN0207_L6.3mm_D2.5mm_P2.54mm_Vertical, F.Cu at (195.8, 85.3)
- added R9: 10k, Resistor_THT:R_Axial_DIN0207_L6.3mm_D2.5mm_P2.54mm_Vertical, F.Cu at (206.1, 80.3)
- renumbered R4 to R5
Connections:
- JP2 pad 1: Net-(J1-Pad6) -> Net-(J2-Pad3)
- JP2 pad 2: /1(Tx) -> Net-(JP2-Pad2)
- JP3 pad 1: Net-(J1-Pad7) -> Net-(J1-Pad6)
- JP3 pad 2: /0(Rx) -> Net-(JP3-Pad2)
- P1 pad 5: (no net) -> +5V
- P3 pad 10: /8 -> (no net)
- P4 pad 1: (no net) -> /7
- P4 pad 2: (no net) -> /6(**)
- R2 pad 2: /1(Tx) -> Net-(JP2-Pad2)
- R3 pad 2: /0(Rx) -> Net-(JP3-Pad2)
- R5 pad 1: /8 -> /7
- R5 pad 2: Net-(JP1-Pad2) -> Net-(Q1-Pad3)

Commit message: add arduino uno sheild pcb
add arduino uno sheild pcb
Parts:
- added JP5: SolderJumper_2_Open, Jumper:SolderJumper-2_P1.3mm_Open_Pad1.0x1.5mm, F.Cu at (167.3, 79.9)
- added JP6: SolderJumper_2_Open, Jumper:SolderJumper-2_P1.3mm_Open_Pad1.0x1.5mm, F.Cu at (163.6, 79.9)
- moved Q2 86.8 mm to (128.5, 102.4), turned to 180 degrees
- moved Q1 80.3 mm to (123.0, 102.4), turned to 180 degrees
- moved R9 76.6 mm to (130.5, 92.4), turned to 270 degrees
- moved Q3 75.9 mm to (134.0, 102.4), turned to 180 degrees
- moved Q4 74.8 mm to (139.5, 102.4), turned to 180 degrees
- moved L1 73.8 mm to (119.0, 83.9), turned to 270 degrees
- moved R10 69.9 mm to (126.0, 92.4), turned to 270 degrees
- moved R5 69.3 mm to (130.7, 82.6), turned to 270 degrees
- moved R1 65.6 mm to (126.0, 111.4), turned to 90 degrees
- moved R6 64.5 mm to (135.5, 82.5), turned to 270 degrees
- moved R3 62.8 mm to (135.0, 111.4), turned to 90 degrees
- moved R8 61.2 mm to (135.0, 92.4), turned to 270 degrees
- moved R2 60.6 mm to (130.5, 111.4), turned to 90 degrees
- moved R4 56.5 mm to (139.5, 111.4), turned to 90 degrees
- moved JP1 51.3 mm to (155.5, 79.9), turned to 90 degrees
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Connections:
- JP1 pad 1: Net-(J2-Pad11) -> Net-(JP1-Pad1)
- JP1 pad 2: Net-(JP1-Pad2) -> /7
- JP2 pad 1: Net-(J2-Pad3) -> Net-(JP2-Pad1)
- JP2 pad 2: Net-(JP2-Pad2) -> /6(**)
- JP3 pad 1: Net-(J1-Pad6) -> Net-(JP3-Pad1)
- JP3 pad 2: Net-(JP3-Pad2) -> /0(Rx)
- JP4 pad 1: Net-(J1-Pad7) -> Net-(JP4-Pad1)
- JP4 pad 2: Net-(JP4-Pad2) -> /1(Tx)
- P4 pad 5: (no net) -> /3(**)
- P4 pad 6: (no net) -> /2
- Q1 pad 2: Net-(JP1-Pad2) -> Net-(J2-Pad11)
- Q2 pad 2: Net-(JP2-Pad2) -> Net-(J2-Pad3)
- Q3 pad 2: Net-(JP3-Pad2) -> Net-(J1-Pad6)
- Q3 pad 3: /0(Rx) -> Net-(JP3-Pad1)
- Q4 pad 2: Net-(JP4-Pad2) -> Net-(J1-Pad7)
- Q4 pad 3: /1(Tx) -> Net-(JP4-Pad1)
- R1 pad 2: Net-(JP1-Pad2) -> Net-(J2-Pad11)
- R2 pad 2: Net-(JP2-Pad2) -> Net-(J2-Pad3)
- R3 pad 2: Net-(JP3-Pad2) -> Net-(J1-Pad6)
- R4 pad 2: Net-(JP4-Pad2) -> Net-(J1-Pad7)
- R5 pad 1: /7 -> Net-(JP1-Pad1)
- R6 pad 1: /6(**) -> Net-(JP2-Pad1)
- R7 pad 2: /1(Tx) -> Net-(JP4-Pad1)
- R8 pad 2: /0(Rx) -> Net-(JP3-Pad1)
Routing:
- net +3V3: track 0.00 -> 125.6 mm
- net /A5(SCL): track 0.00 -> 99.5 mm, vias 0 -> 2
- net /A4(SDA): track 0.00 -> 96.8 mm, vias 0 -> 2
- net GND: track 0.00 -> 96.4 mm, vias 0 -> 14
- net +5V: track 0.00 -> 64.3 mm
- net Net-(JP3-Pad1): track 0.00 -> 62.1 mm
- net Net-(J2-Pad11): track 0.00 -> 55.8 mm, vias 0 -> 2
- net Net-(JP4-Pad1): track 0.00 -> 52.8 mm, vias 0 -> 3
- net Net-(J1-Pad6): track 0.00 -> 51.7 mm
- net Net-(J1-Pad7): track 0.00 -> 42.4 mm
- net Net-(J2-Pad3): track 0.00 -> 38.6 mm
- net Net-(JP1-Pad1): track 0.00 -> 25.7 mm
- net Net-(JP2-Pad1): track 0.00 -> 24.5 mm
- net Net-(Q1-Pad3): track 0.00 -> 20.9 mm
- net Net-(Q2-Pad3): track 0.00 -> 20.6 mm
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- added copper zone on B.Cu, net GND
- added copper zone on F.Cu, net GND
Other:
- board text added: "211124 V1.1 ES920LRB-Arduino_Uno-Shield"
