File: ES920LRB-Arduino_Uno-Shield/ES920LRB-Arduino-Shield.kicad_pcb (KiCad board)
At the start: 2 copper layers, 68.6 x 53.3 mm, 33 parts, among them J1 Conn_01x10_Female, J2 Conn_01x12_Female, M1 ES920LR2B, P1 Power, P2 Analog, P3 Digital, P4 Digital, P5 CONN_01X01, P6 CONN_01X01, P7 CONN_01X01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

Commit message: add arduino uno shield v1.6
add arduino uno shield v1.6
Other:
- board text added: "211124 V1.6 ES920LRB-Arduino_Uno-Shield"
- board text removed: "211124 V1.0 ES920LRB-Arduino_Uno-Shield"
Changed lines of the file:
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@@
     (title ES920LRB-Arduino_Uno-Shield)
     (date 2021-11-24)
-    (rev v1.1)
+    (rev v1.6)
     (company "teTra Aviation Corp.")
   )
@@
   )
   (setup
-    (last_trace_width 1)
+    (last_trace_width 0.25)
     (user_trace_width 0.25)
     (user_trace_width 0.5)
@@
     (visible_elements FFFFFF7F)
     (pcbplotparams
-      (layerselection 0x00030_ffffffff)
-      (usegerberextensions false)
-      (usegerberattributes true)
+      (layerselection 0x010f0_ffffffff)
+      (usegerberextensions true)
+      (usegerberattributes false)
       (usegerberadvancedattributes true)
       (creategerberjobfile true)
@@
     (pad 1 thru_hole circle (at 0 0) (size 4.064 4.064) (drill 3.048) (layers *.Cu *.Mask F.SilkS))
   )
-  (gr_text "211124 V1.0\nES920LRB-Arduino_Uno-Shield" (at 115.998 78.865 270) (layer F.SilkS)
+  (gr_text "211124 V1.6\nES920LRB-Arduino_Uno-Shield" (at 115.998 78.865 -90) (layer F.SilkS)
     (effects (font (size 1 1) (thickness 0.15)) (justify left))
   )

Commit message: order pcb v1.x
order pcb v1.x
Other:
- board text added: "211125 V1.7 ES920LR2B-Arduino_Uno-Shield"
- board text removed: "211124 V1.6 ES920LRB-Arduino_Uno-Shield"
