File: ES920LRB-ESP32/ES920LRB-ESP32.sch (KiCad schematic (older format))
At the start: 2 parts

Commit message: add schematica v1.3
add schematica v1.3
Parts:
- added C1, C2: 10uF, Capacitor_THT:C_Rect_L4.0mm_W2.5mm_P2.50mm, symbol Device:C
- added J1, J2: Conn_01x19_Female, Connector_PinHeader_2.54mm:PinHeader_1x19_P2.54mm_Vertical, symbol Connector:Conn_01x19_Female
- added J3, J4: Conn_01x13_Female, Connector_PinHeader_2.54mm:PinHeader_1x13_P2.54mm_Vertical, symbol Connector:Conn_01x13_Female
- added L1: Logo, teTra:teTra-logo, symbol teTra:Logo
- added R1, R2, R3, R4, R5, R6: 10k, Resistor_THT:R_Axial_DIN0207_L6.3mm_D2.5mm_P7.62mm_Horizontal, symbol Device:R
- M1: renamed from M?; footprint (none) -> teTra:ES92LR2B
- gave numbers to parts that had none: 1
Connections:
- net +3V3: now reaches U1.1 (3V3)
- net +3V3: now also M1.13 (VCC), M1.2 (VCCRF), C1.1, C2.1, J1.1 (Pin_1), J3.13 (Pin_13), J3.2 (Pin_2), R1.1, R2.1, R3.1, R4.1
- net at U1.10 (IO26): now also J1.10 (Pin_10)
- net at U1.11 (IO27): now also J1.11 (Pin_11)
- net at U1.12 (IO14): now also J1.12 (Pin_12)
- net at U1.13 (IO12): now also J1.13 (Pin_13)
- net GND: now reaches U1.14 (GND1)
- net GND: now also M1.1 (VSS), M1.26 (GND), U1.20 (GND3), U1.26 (GND2), C1.2, C2.2, J1.14 (Pin_14), J2.1 (Pin_1), J2.7 (Pin_7), J3.1 (Pin_1), J4.13 (Pin_13)
- net at U1.15 (IO13): now also J1.15 (Pin_15)
- net at U1.16 (SD2): now also J1.16 (Pin_16)
- net at U1.17 (SD3): now also J1.17 (Pin_17)
- net at U1.18 (CMD): now also J1.18 (Pin_18)
- net at U1.19 (EXT_5V): now also J1.19 (Pin_19)
- net at U1.2 (EN): now also J1.2 (Pin_2)
- net at U1.21 (IO23): now also J2.2 (Pin_2)
- net at U1.22 (IO22): now also J2.3 (Pin_3)
- net at U1.23 (TXD0): now also J2.4 (Pin_4)
- net at U1.24 (RXD0): now also J2.5 (Pin_5)
- net at U1.25 (IO21): now also J2.6 (Pin_6), R2.2, R6.2
- net at U1.27 (IO19): now also J2.8 (Pin_8), R1.2, R5.2
- net at U1.28 (IO18): now also J2.9 (Pin_9)
- net at U1.29 (IO5): now also J2.10 (Pin_10)
- net at U1.3 (SENSOR_VP): now also J1.3 (Pin_3)
- net Host_RX-ES920_TX: now reaches M1.8 (USART1_TX/PA9)
- net Host_RX-ES920_TX: now also U1.31 (IO16), J2.12 (Pin_12), J3.8 (Pin_8), R4.2; no longer U1.30 (IO17)
- net at U1.32 (IO4): now also J2.13 (Pin_13)
- net at U1.33 (IO0): now also J2.14 (Pin_14)
- net at U1.34 (IO2): now also J2.15 (Pin_15)
- net at U1.35 (IO15): now also J2.16 (Pin_16)
- net at U1.36 (SD1): now also J2.17 (Pin_17)
- net at U1.37 (SD0): now also J2.18 (Pin_18)
- net at U1.38 (CLK): now also J2.19 (Pin_19)
- net at U1.4 (SENSOR_VN): now also J1.4 (Pin_4)
- net at U1.5 (IO34): now also J1.5 (Pin_5)
- net at U1.6 (IO35): now also J1.6 (Pin_6)
- net at U1.7 (IO32): now also J1.7 (Pin_7)
- net at U1.8 (IO33): now also J1.8 (Pin_8)
- net at U1.9 (IO25): now also J1.9 (Pin_9)
- net at M1.10 (PB8/I2C1_SCL): now also J3.10 (Pin_10)
- net at M1.11 (PB9/I2C1_SDA): now also J3.11 (Pin_11)
- net at M1.12 (PA4/DAC1/ADC4): now also J3.12 (Pin_12)
- net at M1.14 (PA3/USART2_RX): now also J4.1 (Pin_1)
- net at M1.15 (PA2/USART2_TX): now also J4.2 (Pin_2)
- net ES920_WKUP1: now reaches M1.16 (SW_INT/PA0/WKUP1)
- net ES920_WKUP1: now also J4.3 (Pin_3), R5.1
- net at M1.17 (PB6/LPTIM1_ETR): now also J4.4 (Pin_4)
- net at M1.18 (PB5/LPTIM1_IN1): now also J4.5 (Pin_5)
- net at M1.19 (LED_T1/PB12/SPI2_NSS): now also J4.6 (Pin_6)
- net at M1.20 (LED_T0/PB13/SPI2_SCK): now also J4.7 (Pin_7)
- net at M1.21 (PB15/SPI2_MOSI): now also J4.8 (Pin_8)
- net at M1.22 (PB14/SPI2_MISO): now also J4.9 (Pin_9)
- net at M1.23 (PA5/DAC2/ADC5): now also J4.10 (Pin_10)
- net ES920_NRST: now reaches M1.24 (NRST)
- net ES920_NRST: now also J4.11 (Pin_11), R6.1
- net at M1.25 (PB0/ADC8): now also J4.12 (Pin_12)
- net at M1.3 (BOOT0): now also J3.3 (Pin_3)
- net at M1.4 (PC2/ADC12): now also J3.4 (Pin_4)
- net at M1.5 (SWCLK/PA14): now also J3.5 (Pin_5)
- net at M1.6 (SWDIO/PA13): now also J3.6 (Pin_6)
- net at M1.7 (PB11): now also J3.7 (Pin_7)
- net Host_TX-ES920RX: now reaches M1.9 (USART1_RX/PA10)
- net Host_TX-ES920RX: now also U1.30 (IO17), J2.11 (Pin_11), J3.9 (Pin_9), R3.2
Other:
- moved on the sheet: M1, U1

Commit message: add ES920LRB-ESP32 v1.4
add ES920LRB-ESP32 v1.4
Parts:
- added H1, H2, H3, H4: MountingHole, MountingHole:MountingHole_3.2mm_M3, symbol Mechanical:MountingHole
Connections:
- net ES920_NRST: now also R2.2
- net ES920_WKUP1: now also R1.2
- net at J2.6 (Pin_6), R6.2, U1.25 (IO21): no longer R2.2
- net at J2.8 (Pin_8), R5.2, U1.27 (IO19): no longer R1.2
Other:
- moved on the sheet: L1, R5, R6
Changed lines of the file:
@@
 Title "ES920LRB-ESP32"
 Date "2021-11-24"
-Rev "v1.1"
+Rev "v1.3"
 Comp "teTra Aviation Corp."
 Comment1 ""
@@
 	9500 4900 9250 4900
 Wire Wire Line
-	9500 3300 8900 3300
-Wire Wire Line
 	7650 3300 7650 2600
 Wire Wire Line
@@
 L Device:R R5
 U 1 1 61B2AB74
-P 8750 3300
-F 0 "R5" V 8700 3100 50  0000 C CNN
-F 1 "10k" V 8700 3500 50  0000 C CNN
-F 2 "Resistor_THT:R_Axial_DIN0207_L6.3mm_D2.5mm_P7.62mm_Horizontal" V 8680 3300 50  0001 C CNN
-F 3 "~" H 8750 3300 50  0001 C CNN
-	1    8750 3300
-	0    1    1    0
+P 5000 3250
+F 0 "R5" V 4950 3050 50  0000 C CNN
+F 1 "10k" V 4950 3450 50  0000 C CNN
+F 2 "Resistor_THT:R_Axial_DIN0207_L6.3mm_D2.5mm_P7.62mm_Horizontal" V 4930 3250 50  0001 C CNN
+F 3 "~" H 5000 3250 50  0001 C CNN
+	1    5000 3250
+	1    0    0    -1
 $EndComp
 $Comp
 L Device:R R6
 U 1 1 61B2B90E
-P 8750 3400
-F 0 "R6" V 8700 3200 50  0000 C CNN
-F 1 "10k" V 8700 3600 50  0000 C CNN
-F 2 "Resistor_THT:R_Axial_DIN0207_L6.3mm_D2.5mm_P7.62mm_Horizontal" V 8680 3400 50  0001 C CNN
-F 3 "~" H 8750 3400 50  0001 C CNN
-	1    8750 3400
-	0    1    1    0
+P 5300 3250
+F 0 "R6" V 5250 3050 50  0000 C CNN
+F 1 "10k" V 5250 3450 50  0000 C CNN
+F 2 "Resistor_THT:R_Axial_DIN0207_L6.3mm_D2.5mm_P7.62mm_Horizontal" V 5230 3250 50  0001 C CNN
+F 3 "~" H 5300 3250 50  0001 C CNN
+	1    5300 3250
+	1    0    0    -1
 $EndComp
 $Comp
@@
 	5300 2700 7550 2700
 Wire Wire Line
-	8900 3400 9600 3400
-Wire Wire Line
-	8600 3300 7650 3300
-Wire Wire Line
-	7550 3400 8600 3400
-Wire Wire Line
 	5900 2350 5900 4550
 Wire Wire Line
@@
 	5000 1900 5000 2050
 Wire Wire Line
-	5000 2600 5000 4200
-Wire Wire Line
 	5000 4200 4150 4200
-Connection ~ 5000 2600
-Wire Wire Line
-	5300 2700 5300 4000
 Wire Wire Line
 	5300 4000 4150 4000
-Connection ~ 5300 2700
 Wire Wire Line
 	5900 4550 5500 4550
@@
 L teTra:Logo L1
 U 1 1 61CC2BF5
-P 10850 6900
-F 0 "L1" H 11028 7021 50  0000 L CNN
-F 1 "Logo" H 11028 6930 50  0000 L CNN
-F 2 "teTra:teTra-logo" H 10850 6900 50  0001 C CNN
-F 3 "" H 10850 6900 50  0001 C CNN
-	1    10850 6900
+P 10800 6800
+F 0 "L1" H 10978 6921 50  0000 L CNN
+F 1 "Logo" H 10978 6830 50  0000 L CNN
+F 2 "teTra:teTra-logo" H 10800 6800 50  0001 C CNN
+F 3 "" H 10800 6800 50  0001 C CNN
+	1    10800 6800
+	1    0    0    -1
+$EndComp
+$Comp
+L Mechanical:MountingHole H2
+U 1 1 61A0A9D3
+P 9200 6750
+F 0 "H2" H 9300 6796 50  0000 L CNN
+F 1 "MountingHole" H 9300 6705 50  0000 L CNN
+F 2 "MountingHole:MountingHole_3.2mm_M3" H 9200 6750 50  0001 C CNN
+F 3 "~" H 9200 6750 50  0001 C CNN
+	1    9200 6750
+	1    0    0    -1
+$EndComp
+$Comp
+L Mechanical:MountingHole H3
+U 1 1 61A163B5
+P 9950 6750
+F 0 "H3" H 10050 6796 50  0000 L CNN
+F 1 "MountingHole" H 10050 6705 50  0000 L CNN
+F 2 "MountingHole:MountingHole_3.2mm_M3" H 9950 6750 50  0001 C CNN
+F 3 "~" H 9950 6750 50  0001 C CNN
+	1    9950 6750
+	1    0    0    -1
+$EndComp
+$Comp
+L Mechanical:MountingHole H4
+U 1 1 61A1077A
+P 9950 7000
+F 0 "H4" H 10050 7046 50  0000 L CNN
+F 1 "MountingHole" H 10050 6955 50  0000 L CNN
+F 2 "MountingHole:MountingHole_3.2mm_M3" H 9950 7000 50  0001 C CNN
+F 3 "~" H 9950 7000 50  0001 C CNN
+	1    9950 7000
+	1    0    0    -1
+$EndComp
+$Comp
+L Mechanical:MountingHole H1
+U 1 1 61A00C12
+P 9200 7000
+F 0 "H1" H 9300 7046 50  0000 L CNN
+F 1 "MountingHole" H 9300 6955 50  0000 L CNN
+F 2 "MountingHole:MountingHole_3.2mm_M3" H 9200 7000 50  0001 C CNN
+F 3 "~" H 9200 7000 50  0001 C CNN
+	1    9200 7000
 	1    0    0    -1
 $EndComp
@@
 L Graphic:SYM_Radio_Waves_Small #SYM1
 U 1 1 61CC4447
-P 10450 6800
-F 0 "#SYM1" H 10450 6940 50  0001 C CNN
-F 1 "SYM_Radio_Waves_Small" H 10450 6675 50  0001 C CNN
-F 2 "" H 10450 6625 50  0001 C CNN
-F 3 "~" H 10480 6600 50  0001 C CNN
-	1    10450 6800
-	1    0    0    -1
-$EndComp
+P 10800 7000
+F 0 "#SYM1" H 10800 7140 50  0001 C CNN
+F 1 "SYM_Radio_Waves_Small" H 10800 6875 50  0001 C CNN
+F 2 "" H 10800 6825 50  0001 C CNN
+F 3 "~" H 10830 6800 50  0001 C CNN
+	1    10800 7000
+	1    0    0    -1
+$EndComp
+Wire Wire Line
+	5300 2700 5300 3100
+Connection ~ 5300 2700
+Wire Wire Line
+	5300 3400 5300 4000
+Wire Wire Line
+	5000 3400 5000 4200
+Wire Wire Line
+	5000 3100 5000 2600
+Connection ~ 5000 2600
+Wire Wire Line
+	7650 3300 9500 3300
+Wire Wire Line
+	7550 3400 9600 3400
 $EndSCHEMATC
